File: hardware/ws2812_tester/ws2812_tester.kicad_sch (KiCad schematic)
At the start: 0 parts

Commit message: Adds first version of the schematics
Parts:
- added C1: 1µF, symbol Device:C_Small
- added C2: 100nF, symbol Device:C_Small
- added F1: 1A, symbol Device:Polyfuse_Small
- added J1: USB_C_DEALON-USB-US31-106, ws2812_tester:DEALON_USB-US31-106, symbol ws2812_tester:USB_C_DEALON-USB-US31-106
- added J2: Pins_1-4, symbol Connector_Generic:Conn_01x04
- added J3: Conn_01x03, symbol Connector_Generic:Conn_01x03
- added J4: Pins_5-8, symbol Connector_Generic:Conn_01x04
- added Q1: PMN48XP, Package_SO:TSOP-6_1.65x3.05mm_P0.95mm, symbol Transistor_FET:PMN48XP
- added R1, R2: 5.1kΩ, symbol Device:R_Small_US
- added R3: 10kΩ, symbol Device:R_Small_US
- added U1: ATtiny85-20S, Package_SO:SOIC-8W_5.3x5.3mm_P1.27mm, symbol MCU_Microchip_ATtiny:ATtiny85-20S
Connections:
- new net: J1.A5 (CC1), R1.1
- new net: J1.B5 (CC2), R2.1
- new net: F1.2, Q1.1 (D), Q1.2 (D), Q1.5 (D), Q1.6 (D)
- new net +5V: F1.1, J1.A9 (VBUS), J1.B9 (VBUS), J3.3 (Pin_3)
- new net GND: C1.2, C2.2, J1.A12 (GND), J1.B12 (GND), J1.S1 (SHIELD), J2.4 (Pin_4), J3.1 (Pin_1), Q1.3 (G), R1.2, R2.2, U1.4 (GND)
- new net PB0: J4.4 (Pin_4), U1.5 (AREF/PB0)
- new net PB1/LED_DATA: J3.2 (Pin_2), J4.3 (Pin_3), U1.6 (PB1)
- new net PB2: J4.2 (Pin_2), U1.7 (PB2)
- new net PB3: J2.2 (Pin_2), U1.2 (XTAL1/PB3)
- new net PB4: J2.3 (Pin_3), U1.3 (XTAL2/PB4)
- new net PB5/RST: J2.1 (Pin_1), R3.2, U1.1 (~{RESET}/PB5)
- new net VCC: C1.1, C2.1, J4.1 (Pin_1), Q1.4 (S), R3.1, U1.8 (VCC)
Other:
- note added: "Connectors"
- note added: "Microcontroller"
- note added: "Power protection"
